File: BlackPanda/kicad_project/BlackPanda.kicad_sch (KiCad schematic)
At the start: 86 parts, among them P1 TYPE-C-31-M-04, Q1 DDTA143ECA-7-F P08, Q2 DDTA143ECA-7-F P08, Q3 PDTC114EU, Q4 HY12P03C2, SW1 SW_Push, U1 AP22615AWU-7, U10 TJA1042TK-3, U11 TJA1042TK-3, U12 XL1509-3.3, U2 SiP32431DR3, U3 10_0_QHHTZB6_3, U4 NEO-M8M, U5 FM-B1921RGBA-SH, U6 TPS5450DDAR, U7 STM32F413RGTx, U8 TJA1042TK-3, U9 TJA1042TK-3, Y1 X322516MLB4SI

Commit message: TJA1042 uses HVSON8
Parts:
- U10, U11, U8, U9: footprint Package_DFN_QFN:DFN-8-1EP_3x3mm_P0.65mm_EP1.55x2.4mm -> Package_SON:HVSON-8-1EP_3x3mm_P0.65mm_EP1.6x2.4mm
Changed lines of the file:
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@@
       (effects (font (size 1.27 1.27)) (justify left))
     )
-    (property "Footprint" "Package_DFN_QFN:DFN-8-1EP_3x3mm_P0.65mm_EP1.55x2.4mm" (at 450.85 185.42 0)
+    (property "Footprint" "Package_SON:HVSON-8-1EP_3x3mm_P0.65mm_EP1.6x2.4mm" (at 450.85 185.42 0)
       (effects (font (size 1.27 1.27) italic) hide)
     )
@@
       (effects (font (size 1.27 1.27)) (justify left))
     )
-    (property "Footprint" "Package_DFN_QFN:DFN-8-1EP_3x3mm_P0.65mm_EP1.55x2.4mm" (at 452.12 287.02 0)
+    (property "Footprint" "Package_SON:HVSON-8-1EP_3x3mm_P0.65mm_EP1.6x2.4mm" (at 452.12 287.02 0)
       (effects (font (size 1.27 1.27) italic) hide)
     )
@@
       (effects (font (size 1.27 1.27)) (justify left))
     )
-    (property "Footprint" "Package_DFN_QFN:DFN-8-1EP_3x3mm_P0.65mm_EP1.55x2.4mm" (at 452.12 336.55 0)
+    (property "Footprint" "Package_SON:HVSON-8-1EP_3x3mm_P0.65mm_EP1.6x2.4mm" (at 452.12 336.55 0)
       (effects (font (size 1.27 1.27) italic) hide)
     )
@@
       (effects (font (size 1.27 1.27)) (justify left))
     )
-    (property "Footprint" "Package_DFN_QFN:DFN-8-1EP_3x3mm_P0.65mm_EP1.55x2.4mm" (at 452.12 237.49 0)
+    (property "Footprint" "Package_SON:HVSON-8-1EP_3x3mm_P0.65mm_EP1.6x2.4mm" (at 452.12 237.49 0)
       (effects (font (size 1.27 1.27) italic) hide)
     )
